File: pcb-ehd/integrated-pcb/blinky-bowtie.kicad_pcb (KiCad board)
At the start: 2 copper layers, 91 parts, among them J1 USB_C_Receptacle_USB2.0, J2 JST_PH, J3 SWD, Q1 DMP2045U, SW1 B3U, SW2 B3U, SW3 B3U, U1 MCP73831T-2, U2 ATSAMD21G18A-M, U3 AP2112K-3.3, U4 MAX9814, U5 W25Q32JVZPIQ

Commit message: bow tie graphics done
Parts:
- added C37: 1u, Capacitor_SMD:C_0603_1608Metric, F.Cu at (-50.7, 50.4)
- added LOGO1: F.Silk, ehd:bowtie-f-silk, F.Cu at (154.6, 113.9)
- added LOGO2: Edge.Cuts, ehd:bowtie-edge-cuts, F.Cu at (156.4, 112.4)
- added R14: 10K, Resistor_SMD:R_0603_1608Metric, F.Cu at (-50.7, 52.9)
- added SW4: SLIDE, ehd:SW_SPDT_PCM12, F.Cu at (-57.6, 52.1)
- added U6: SN74LVC1T45DCK, Package_TO_SOT_SMD:SOT-363_SC-70-6, F.Cu at (-150.7, 39.7)
- moved C10 289.2 mm to (-150.8, 47.9)
- moved C33 284.7 mm to (-142.4, 35.0)
- moved C29 281.2 mm to (-142.4, 32.4)
- moved C30 277.0 mm to (-133.9, 25.8)
- moved C7 276.9 mm to (-138.3, 32.4)
- moved C9 273.4 mm to (-146.5, 39.1)
- moved C8 272.9 mm to (-138.3, 35.0)
- moved C17 270.6 mm to (-150.8, 42.9)
- moved D11 267.6 mm to (-140.2, 27.9)
- moved D24 266.2 mm to (-148.6, 14.6)
- moved C18 265.4 mm to (-133.9, 30.8)
- moved D10 259.6 mm to (-148.6, 21.3)
- moved C5 256.9 mm to (-117.1, 12.6)
- moved C23 255.2 mm to (-146.5, 41.6)
- moved C16 254.7 mm to (-150.8, 45.4)
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Connections:
- C21 pad 1: +3V3 -> Net-(C21-Pad1)
- D25 pad 2: (no net) -> unconnected-(D25-Pad2)
- D6 pad 4: (no net) -> Net-(D6-Pad4)
- FB1 pad 2: Net-(FB1-Pad2) -> Net-(C21-Pad1)
- U4 pad 2: Net-(FB1-Pad2) -> Net-(C21-Pad1)
- U4 pad 5: Net-(FB1-Pad2) -> Net-(C21-Pad1)
Other:
- board outline added: 142.7 x 72 mm

Commit message: rough placement of all but analog
Parts:
- C1, C10, C11, C12, C13, C14, C15, C16, C17, C18, C19, C2, C20, C21, C22, C23, C24, C25, C26, C27, C28, C29, C3, C30, C31, C32, C33, C34, C35, C36, C37, C4, C5, C6, C7, C8, C9, D1, D2, D4, D5, FB1, FB2, J1, J2, J3, JP1, JP2, Q1, R1, R10, R11, R12, R13, R14, R2, R3, R4, R5, R6, R7, R8, R9, SW1, SW2, SW3, SW4, U1, U2, U3, U4, U5, U6: moved to B.Cu
- D10, D11, D12, D13, D14, D15, D16, D17, D18, D19, D20, D21, D22, D23, D24, D25, D6, D7, D8, D9: footprint LED_SMD:LED_WS2812B_PLCC4_5.0x5.0mm_P3.2mm -> ehd:LED_WS2812B_PLCC4_5.0x5.0mm_P3.2mm
- D3: footprint LED_SMD:LED_WS2812B_PLCC4_5.0x5.0mm_P3.2mm -> ehd:LED_WS2812B_PLCC4_5.0x5.0mm_P3.2mm; moved to B.Cu
- moved D24 380.7 mm to (220.4, 108.5)
- moved C29 370.6 mm to (220.4, 108.5)
- moved D25 361.3 mm to (216.4, 124.4)
- moved C30 358.7 mm to (218.7, 91.3)
- moved D22 355.9 mm to (216.4, 75.5)
- moved D18 355.7 mm to (188.5, 114.9)
- moved D21 354.5 mm to (202.4, 78.0)
- moved C31 351.8 mm to (214.7, 75.5)
- moved D23 347.1 mm to (220.4, 91.3)
- moved C33 345.8 mm to (200.7, 78.0)
- moved C32 345.5 mm to (220.4, 104.5)
- moved C26 345.0 mm to (214.7, 124.4)
- moved D19 337.1 mm to (202.4, 121.9)
- moved D20 336.7 mm to (202.4, 100.0)
- moved D16 331.6 mm to (176.4, 100.0)
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Connections:
- D3 pad 2: (no net) -> unconnected-(D3-Pad2)
- U6 pad 3: /LEDs/LEDS -> (no net)
- U6 pad 5: /LEDs/LEDS -> +3V3
Routing:
- net /D-: track 0.00 -> 20.4 mm
- net /D+: track 0.00 -> 18.9 mm
Other:
- board text added: "3V3"
- board text added: "CHARGE"
- board text added: "LiPo lives here!"
- board text added: "USER"

Commit message: layout passes DRC
Parts:
- added H1: M2, MountingHole:MountingHole_2.2mm_M2_DIN965, F.Cu at (146.2, 109.6)
- added H2: M2, MountingHole:MountingHole_2.2mm_M2_DIN965, F.Cu at (164.2, 109.6)
- added H3: M2, MountingHole:MountingHole_2.2mm_M2_DIN965, F.Cu at (164.2, 91.6)
- added H4: M2, MountingHole:MountingHole_2.2mm_M2_DIN965, F.Cu at (146.2, 91.6)
- moved R11 41.5 mm to (159.3, 107.7), turned to 90 degrees
- moved JP2 37.5 mm to (138.8, 106.7), turned to 0 degrees
- moved JP1 35.9 mm to (138.8, 104.1), turned to 0 degrees
- moved R12 34.8 mm to (160.8, 107.7), turned to -90 degrees
- moved U4 34.1 mm to (155.0, 106.1), turned to 0 degrees
- moved FB1 31.0 mm to (150.5, 103.5), turned to 0 degrees
- moved R10 30.9 mm to (160.0, 110.0), turned to 0 degrees
- moved C27 30.2 mm to (150.5, 108.0), turned to 0 degrees
- moved C34 29.9 mm to (160.0, 105.4), turned to 0 degrees
- moved C21 29.4 mm to (150.5, 105.0)
- moved C28 27.6 mm to (156.5, 101.8), turned to -90 degrees
- moved C35 25.6 mm to (150.5, 106.5)
- moved FB2 19.7 mm to (148.2, 100.8)
- moved R3 0.49 mm to (100.4, 80.2)
- moved R5 0.49 mm to (101.9, 80.2)
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Connections:
- D25 pad 2: unconnected-(D25-Pad2) -> (no net)
- D3 pad 2: unconnected-(D3-Pad2) -> (no net)
- JP1 pad 1: (no net) -> /A0
- JP2 pad 1: (no net) -> /A2
- SW1 pad 1: (no net) -> /D1
- SW3 pad 1: (no net) -> /SCK
- U2 pad 15: (no net) -> /D1
- U2 pad 20: (no net) -> /SCK
- U2 pad 24: (no net) -> /D5
- U2 pad 3: (no net) -> /A0
- U2 pad 8: (no net) -> /A2
- U6 pad 3: (no net) -> /D5
Routing:
- net +3V3: track 0.00 -> 247.1 mm, vias 0 -> 15
- net +5V: track 0.00 -> 174.4 mm, vias 0 -> 4
- net /D9: track 0.00 -> 164.2 mm, vias 0 -> 2
- net /D13: track 0.00 -> 154.0 mm, vias 0 -> 6
- net VCC: track 0.00 -> 84.3 mm, vias 0 -> 24
- net +BATT: track 0.00 -> 60.3 mm
- net Net-(D15-Pad2): track 0.00 -> 55.3 mm, vias 0 -> 2
- net GND: track 0.00 -> 51.1 mm, vias 0 -> 62
- net /A2: track 0.00 -> 47.8 mm, vias 0 -> 2
- net /nRST: track 0.00 -> 46.2 mm, vias 0 -> 2
- net /A0: track 0.00 -> 45.6 mm, vias 0 -> 2
- net /GAIN: track 0.00 -> 36.3 mm, vias 0 -> 2
- net /AR: track 0.00 -> 35.9 mm, vias 0 -> 2
- net /D1: track 0.00 -> 34.2 mm, vias 0 -> 4
- net Net-(D14-Pad2): track 0.00 -> 32.7 mm, vias 0 -> 2
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- added copper zone on F.Cu, net GND
- added copper zone on F.Cu, net GNDA
- added copper zone on B.Cu, net VCC
Other:
- board text added: "AR"
- board text added: "Blinky Bowtie BSides CBR 2021"
- board text added: "GAIN"
- board text added: "GND"
- board text added: "Josh Johnson @_joshajohnson"
- board text added: "OFF"
- board text added: "ON"
- board text added: "Place in OFF before connecting USB"
- board text added: "RESET"
- board text added: "SW0"
- board text added: "SW1"
- board text added: "SWD CLK"
- board text added: "SWD IO"
- board text added: "nRST"

Commit message: updates with ordering
Routing:
- net /D9: track 164.2 -> 160.4 mm
- net +3V3: track 247.1 -> 249.0 mm
- net /D13: track 154.0 -> 155.8 mm
- net +5V: track 174.4 -> 175.0 mm
Other:
- board text added: "JLCJLCJLC"
