File: pcb-ehd/integrated-pcb/blinky-bowtie.kicad_sch (KiCad schematic)
At the start: 60 parts, among them J1 USB_C_Receptacle_USB2.0, J2 JST_PH, J3 SWD, Q1 DMP2045U, SW1 B3U, SW2 B3U, SW3 B3U, SW4 SLIDE, U1 MCP73831T-2, U2 ATSAMD21G18A-M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

Commit message: updates with ordering
Parts:
- D2: LCSC C375450 -> (none); MPN E6C0603SEAC1UDA -> (none); MPN2 Any -> (none); Manufacturer EKINGLUX -> (none); Manufacturer2 Any -> (none)
- U5: LCSC C571260 -> (none); MPN W25Q32JVZPIQ -> (none)
Changed lines of the file:
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@@
       (effects (font (size 1.27 1.27)) hide)
     )
-    (property "LCSC" "C375450" (id 4) (at 21.59 148.59 0)
-      (effects (font (size 1.27 1.27)) hide)
-    )
-    (property "MPN" "E6C0603SEAC1UDA" (id 5) (at 21.59 148.59 0)
-      (effects (font (size 1.27 1.27)) hide)
-    )
-    (property "MPN2" "Any" (id 6) (at 21.59 148.59 0)
-      (effects (font (size 1.27 1.27)) hide)
-    )
-    (property "Manufacturer" "EKINGLUX" (id 7) (at 21.59 148.59 0)
-      (effects (font (size 1.27 1.27)) hide)
-    )
-    (property "Manufacturer2" "Any" (id 8) (at 21.59 148.59 0)
+    (property "LCSC" "" (id 4) (at 21.59 148.59 0)
+      (effects (font (size 1.27 1.27)) hide)
+    )
+    (property "MPN" "" (id 5) (at 21.59 148.59 0)
+      (effects (font (size 1.27 1.27)) hide)
+    )
+    (property "MPN2" "" (id 6) (at 21.59 148.59 0)
+      (effects (font (size 1.27 1.27)) hide)
+    )
+    (property "Manufacturer" "" (id 7) (at 21.59 148.59 0)
+      (effects (font (size 1.27 1.27)) hide)
+    )
+    (property "Manufacturer2" "" (id 8) (at 21.59 148.59 0)
       (effects (font (size 1.27 1.27)) hide)
     )
@@
       (effects (font (size 1.27 1.27)) hide)
     )
-    (property "LCSC" "C571260" (id 4) (at 270.51 151.13 0)
-      (effects (font (size 1.27 1.27)) hide)
-    )
-    (property "MPN" "W25Q32JVZPIQ" (id 5) (at 270.51 151.13 0)
-      (effects (font (size 1.27 1.27)) hide)
-    )
+    (property "LCSC" "" (id 4) (at 270.51 151.13 0)
+      (effects (font (size 1.27 1.27)) hide)
+    )
+    (property "MPN" "" (id 5) (at 270.51 151.13 0)
+      (effects (font (size 1.27 1.27)) hide)
+    )

Commit message: cleanup kicad files
Parts:
- D1: LCSC (none) -> C2286; MPN (none) -> KT-0603R; Manufacturer (none) -> Hubei KENTO Elec
- D2: LCSC (none) -> C375450; MPN (none) -> E6C0603SEAC1UDA; Manufacturer (none) -> EKINGLUX
- D3: LCSC (none) -> C114586; MPN (none) -> WS2812B-B; Manufacturer (none) -> Worldsemi
- D4: LCSC (none) -> C72041; MPN (none) -> 19-217/BHC-ZL1M2RY/3T; Manufacturer (none) -> Everlight Elec
- D5: MPN2 B5817WL -> (none); Manufacturer2 Shikues -> (none)
- FB1, FB2: LCSC (none) -> C76884; MPN (none) -> BLM15AG601SN1D; Manufacturer (none) -> Murata Electronics
- H1, H2, H3, H4, J3, JP1, JP2: DNP (none) -> DNP; now left out of the parts list
- J1: MPN TYPE-C-31-M-12 -> TYPE-C-31-M-12; MPN2 USB4105-GF-A -> (none); Manufacturer Korean Hroparts Elec -> Korean Hroparts Elec; Manufacturer2 GCT -> (none)
- J2: MPN2 C47647 -> (none); Manufacturer2 BOOMELE(Boom Precision Elec) -> (none)
- LOGO1, LOGO2: DNP (none) -> DNP
- MK1: MPN (none) -> MIC_CMA-4544PF-W; Manufacturer (none) -> CUI Devices
- Q1: MPN2 DMP2170U-7 -> (none); Manufacturer2 Diodes Incorporated -> (none)
- SW1, SW2, SW3: LCSC (none) -> C231329; MPN (none) -> B3U-1000P; Manufacturer (none) -> Omron Electronics
- SW4: LCSC (none) -> C221841; MPN (none) -> PCM12SMTR; Manufacturer (none) -> C&K
- U2: LCSC (none) -> C1338342; MPN (none) -> ATSAMD21G18A-MF; Manufacturer (none) -> Microchip Tech
- U3: MPN2 AP7365-33WG-7 -> (none); Manufacturer2 Diodes Incorporated -> (none)
- U4: LCSC (none) -> C41714; MPN (none) -> MAX9814ETD+T; Manufacturer (none) -> Maxim
- U5: value W25Q32JVZPIQ -> GD25Q16CSIGR; LCSC (none) -> C395505; MPN (none) -> GD25Q16CSIGR; Manufacturer Winbond -> Gigadevices
