File: pcb-ehd/module-pcb/module-pcb.kicad_pcb (KiCad board)
At the start: 2 copper layers, 100 x 100 mm, 29 parts, among them J1 Mic-Breakout, J2 Feather

Commit message: updates with ordering
Routing:
- net GND: track 27.5 -> 28.8 mm
Other:
- board text added: "JLCJLCJLCJLC"
Changed lines of the file:
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@@
   )
   (gr_circle (center 100 100) (end 150 100) (layer "Edge.Cuts") (width 0.05) (fill none))
+  (gr_text "JLCJLCJLCJLC" (at 99.999999 55.4) (layer "B.SilkS")
+    (effects (font (size 1 1) (thickness 0.15)) (justify mirror))
+  )
   (gr_text "50dB" (at 101.7 103.9 90) (layer "B.SilkS")
     (effects (font (size 1 1) (thickness 0.15)) (justify mirror))
@@
   (segment (start 65 127.6) (end 65 126.6) (width 0.4) (layer "F.Cu") (net 1))
   (segment (start 54.5 103.8) (end 55.5625 103.8) (width 0.4) (layer "F.Cu") (net 1))
+  (segment (start 57.560641 122.339359) (end 57 122.9) (width 0.25) (layer "F.Cu") (net 1))
   (segment (start 103.8 145.5) (end 103.8 144.4375) (width 0.4) (layer "F.Cu") (net 1))
   (segment (start 98.4 147.45) (end 98.4 148.7) (width 0.4) (layer "F.Cu") (net 1))
@@
   (segment (start 74.1 141.4) (end 74.1 141.081121) (width 0.4) (layer "F.Cu") (net 1))
   (segment (start 96.1 55.5625) (end 96.1 54.4) (width 0.4) (layer "F.Cu") (net 1))
+  (segment (start 58.108238 122.339359) (end 57.560641 122.339359) (width 0.25) (layer "F.Cu") (net 1))
   (segment (start 141.891762 77.660641) (end 142.339359 77.660641) (width 0.4) (layer "F.Cu") (net 1))
   (segment (start 58.6 74.2) (end 59.018879 74.2) (width 0.4) (layer "F.Cu") (net 1))
