File: pcb-ehd/module-pcb/module-pcb.kicad_sch (KiCad schematic)
At the start: 29 parts, among them J1 Mic-Breakout, J2 Feather

Commit message: cleanup kicad files
Parts:
- H1, H2, JP1: DNP (none) -> DNP
Changed lines of the file:
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@@
+      (effects (font (size 1.27 1.27)) hide)
+    )
+    (property "DNP" "DNP" (id 4) (at 54.61 113.665 0)
       (effects (font (size 1.27 1.27)) hide)
     )
@@
       (effects (font (size 1.27 1.27)) hide)
     )
+    (property "DNP" "DNP" (id 4) (at 54.61 118.745 0)
+      (effects (font (size 1.27 1.27)) hide)
+    )
   )
   (symbol (lib_id "Device:C") (at 133.35 71.12 90) (unit 1)
@@
       (effects (font (size 1.27 1.27)) hide)
     )
+    (property "DNP" "DNP" (id 4) (at 55.88 88.9 0)
+      (effects (font (size 1.27 1.27)) hide)
+    )
