File: pcb-sao-magpie/swooping.kicad_pcb (KiCad board)
At the start: 2 copper layers, 49 x 36.6 mm, 12 parts, among them J1 SAO, U1 555

Commit message: cleanup kicad files
Parts:
- removed G***: LOGO, drawing:F.SilkS_g33
- removed G***: LOGO, drawing:F.Mask_g37
- R3: value 470R -> 330R
