File: pcb-sao-magpie/swooping.sch (KiCad schematic (older format))
At the start: 10 parts, among them J1 SAO, U1 555

Commit message: cleanup kicad files
Parts:
- C1: MPN (none) -> CL31B105KOFNNNE; Manufacturer (none) -> Samsung Electro-Mechanics
- D1: MPN (none) -> L513SRD-C; Manufacturer (none) -> American Opto Plus LED
- J1: MPN (none) -> 10129382-904001BLF; Manufacturer (none) -> Amphenol ICC (FCI)
- LOGO1, LOGO2, LOGO4: DNP (none) -> DNP
- R1: MPN (none) -> RMCF1206JT1K00; Manufacturer (none) -> Stackpole Electronics Inc
- R2: MPN (none) -> RMCF1206JT470K; Manufacturer (none) -> Stackpole Electronics Inc
- R3: MPN (none) -> RMCF1206JT330R; Manufacturer (none) -> Stackpole Electronics Inc
- U1: MPN (none) -> TLC555; Manufacturer (none) -> Texas Instruments
Changed lines of the file:
@@
 F 2 "josh-logos:josh-details" H 5900 7200 50  0001 C CNN
 F 3 "~" H 5900 7200 50  0001 C CNN
+F 4 "DNP" H 5900 7200 50  0001 C CNN "DNP"
 	1    5900 7200
 	1    0    0    -1
@@
 F 2 "josh-logos:josh-johnson-logo-8_6x1_5" H 5900 7650 50  0001 C CNN
 F 3 "~" H 5900 7650 50  0001 C CNN
+F 4 "DNP" H 5900 7650 50  0001 C CNN "DNP"
 	1    5900 7650
 	1    0    0    -1
@@
 F 2 "Resistor_SMD:R_1206_3216Metric_Pad1.42x1.75mm_HandSolder" V 4580 3000 50  0001 C CNN
 F 3 "~" H 4650 3000 50  0001 C CNN
+F 4 "RMCF1206JT1K00 " H 4650 3000 50  0001 C CNN "MPN"
+F 5 "Stackpole Electronics Inc" H 4650 3000 50  0001 C CNN "Manufacturer"
 	1    4650 3000
 	1    0    0    -1
@@
 F 2 "Resistor_SMD:R_1206_3216Metric_Pad1.42x1.75mm_HandSolder" V 4580 3400 50  0001 C CNN
 F 3 "~" H 4650 3400 50  0001 C CNN
+F 4 "RMCF1206JT470K" H 4650 3400 50  0001 C CNN "MPN"
+F 5 "Stackpole Electronics Inc" H 4650 3400 50  0001 C CNN "Manufacturer"
 	1    4650 3400
 	1    0    0    -1
@@
 F 2 "Resistor_SMD:R_1206_3216Metric_Pad1.42x1.75mm_HandSolder" V 5780 3600 50  0001 C CNN
 F 3 "~" H 5850 3600 50  0001 C CNN
+F 4 "RMCF1206JT330R" H 5850 3600 50  0001 C CNN "MPN"
+F 5 "Stackpole Electronics Inc" H 5850 3600 50  0001 C CNN "Manufacturer"
 	1    5850 3600
 	1    0    0    -1
@@
 F 2 "LED_THT:LED_D5.0mm" H 5850 3950 50  0001 C CNN
 F 3 "~" H 5850 3950 50  0001 C CNN
+F 4 "L513SRD-C" H 5850 3950 50  0001 C CNN "MPN"
+F 5 "American Opto Plus LED" H 5850 3950 50  0001 C CNN "Manufacturer"
 	1    5850 3950
 	0    -1   -1   0
@@
 F 2 "Capacitor_SMD:C_1206_3216Metric_Pad1.42x1.75mm_HandSolder" H 4688 3650 50  0001 C CNN
 F 3 "~" H 4650 3800 50  0001 C CNN
+F 4 "CL31B105KOFNNNE" H 4650 3800 50  0001 C CNN "MPN"
+F 5 "Samsung Electro-Mechanics" H 4650 3800 50  0001 C CNN "Manufacturer"
 	1    4650 3800
 	1    0    0    -1
@@
 F 2 "Connector_PinHeader_2.54mm:PinHeader_2x02_P2.54mm_Vertical" H 6950 3750 50  0001 C CNN
 F 3 "" H 6950 3750 50  0001 C CNN
+F 4 "10129382-904001BLF" H 6950 3600 50  0001 C CNN "MPN"
+F 5 "Amphenol ICC (FCI)" H 6950 3600 50  0001 C CNN "Manufacturer"
 	1    6950 3600
 	1    0    0    -1
@@
 F 2 "josh-logos:OSHW_Logo_3.6x3.6_F.Mask" H 6450 7500 50  0001 C CNN
 F 3 "~" H 6450 7500 50  0001 C CNN
+F 4 "DNP" H 6450 7500 50  0001 C CNN "DNP"
 	1    6450 7500
 	1    0    0    -1
@@
 F 2 "Package_SO:SOIC-8_3.9x4.9mm_P1.27mm" H 5400 3650 50  0001 C CNN
 F 3 "" H 5400 3650 50  0001 C CNN
+F 4 "TLC555" H 5400 3400 50  0001 C CNN "MPN"
+F 5 "Texas Instruments" H 5400 3400 50  0001 C CNN "Manufacturer"
 	1    5400 3400
 	1    0    0    -1
